Commit message: ported ros1 package structure

File: ezgripper_description/urdf/ezgripper_single_mount.urdf.xacro (robot description, xacro)
@@ -1,5 +1,5 @@
 <?xml version="1.0" encoding="UTF-8"?>
-<robot name="ezgripper_dual_gen2_single_mount" xmlns:xacro="http://ros.org/wiki/xacro">
-	<xacro:macro name="ezgripper_dual_gen2_single_mount" params="prefix parent_link *origin">
+<robot name="ezgripper_single_mount" xmlns:xacro="http://ros.org/wiki/xacro">
+	<xacro:macro name="ezgripper_single_mount" params="prefix parent_link *origin">
 		<!-- links -->
 		<link name="${prefix}_ezgripper_mount">
@@ -7,5 +7,5 @@
 				<xacro:insert_block name="origin"/>
 				<geometry>
-					<mesh filename="file://$(find ezgripper_description)/meshes/dual_gen2_single_mount/SAKE_Single_Mount.stl"/>
+					<mesh filename="file://$(find ezgripper_description)/meshes/visual/SAKE_Single_Mount.stl"/>
 				</geometry>
 				<material name="blue"/>
@@ -14,5 +14,5 @@
 				<xacro:insert_block name="origin"/>
 				<geometry>
-					<mesh filename="file://$(find ezgripper_description)/meshes/dual_gen2_single_mount/SAKE_Single_Mount.stl"/>
+					<mesh filename="file://$(find ezgripper_description)/meshes/collision/SAKE_Single_Mount.stl"/>
 				</geometry>
 			</collision>
@@ -41,5 +41,5 @@
 				<origin xyz="0.0 0 0" rpy="0 0 0"/>
 				<geometry>
-					<mesh filename="file://$(find ezgripper_description)/meshes/dual_gen2_single_mount/SAKE_Palm_IM.stl"/>
+					<mesh filename="file://$(find ezgripper_description)/meshes/visual/SAKE_Palm_IM.stl"/>
 				</geometry>
 				<material name="blue"/>
@@ -48,5 +48,5 @@
 				<origin xyz="0.0 0 0" rpy="0 0 0"/>
 				<geometry>
-					<mesh filename="file://$(find ezgripper_description)/meshes/dual_gen2_single_mount/SAKE_Palm_IM.stl"/>
+					<mesh filename="file://$(find ezgripper_description)/meshes/collision/SAKE_Palm_IM.stl"/>
 				</geometry>
 			</collision>
@@ -88,5 +88,5 @@
 				<origin xyz="0 0 0" rpy="0 0 0"/>
 				<geometry>
-					<mesh filename="file://$(find ezgripper_description)/meshes/dual_gen2_single_mount/SAKE_Finger_L1_IM.stl"/>
+					<mesh filename="file://$(find ezgripper_description)/meshes/visual/SAKE_Finger_L1_IM.stl"/>
 				</geometry>
 				<material name="grey"/>
@@ -95,5 +95,5 @@
 				<origin xyz="0 0 0" rpy="0 0 0"/>
 				<geometry>
-					<mesh filename="file://$(find ezgripper_description)/meshes/dual_gen2_single_mount/SAKE_Finger_L1_IM.stl"/>
+					<mesh filename="file://$(find ezgripper_description)/meshes/collision/SAKE_Finger_L1_IM.stl"/>
 				</geometry>
 			</collision>
@@ -112,5 +112,5 @@
 				<origin xyz="0 0 0" rpy="0 0 0"/>
 				<geometry>
-					<mesh filename="file://$(find ezgripper_description)/meshes/dual_gen2_single_mount/SAKE_Finger_L2_IM.stl"/>
+					<mesh filename="file://$(find ezgripper_description)/meshes/visual/SAKE_Finger_L2_IM.stl"/>
 				</geometry>
 				<material name="grey"/>
@@ -119,5 +119,5 @@
 				<origin xyz="0 0 0" rpy="0 0 0"/>
 				<geometry>
-					<mesh filename="file://$(find ezgripper_description)/meshes/dual_gen2_single_mount/SAKE_Finger_L2_IM.stl"/>
+					<mesh filename="file://$(find ezgripper_description)/meshes/collision/SAKE_Finger_L2_IM.stl"/>
 				</geometry>
 			</collision>
@@ -136,5 +136,5 @@
 				<origin xyz="0 0 0" rpy="0 0 0"/>
 				<geometry>
-					<mesh filename="file://$(find ezgripper_description)/meshes/dual_gen2_single_mount/SAKE_Finger_Pad_IM.stl"/>
+					<mesh filename="file://$(find ezgripper_description)/meshes/visual/SAKE_Finger_Pad_IM.stl"/>
 				</geometry>
 				<material name="grey"/>
@@ -143,5 +143,5 @@
 				<origin xyz="0 0 0" rpy="0 0 0"/>
 				<geometry>
-					<mesh filename="file://$(find ezgripper_description)/meshes/dual_gen2_single_mount/SAKE_Finger_Pad_IM.stl"/>
+					<mesh filename="file://$(find ezgripper_description)/meshes/collision/SAKE_Finger_Pad_IM.stl"/>
 				</geometry>
 			</collision>
@@ -227,10 +227,10 @@
 		<plugin name="gazebo_ros2_control" filename="libgazebo_ros2_control.so">
 			<ros>
-				<namespace>/ezgripper_dual_gen2_single_mount</namespace>
+				<namespace>/ezgripper_single_mount</namespace>
 			</ros>
 			<robot_param>robot_description</robot_param>
       <robot_param_node>/robot_state_publisher</robot_param_node>
 			<robot_sim_type>gazebo_ros2_control/GazeboSystem</robot_sim_type>
-			<parameters>$(find ezgripper_control)/config/controllers_dual_gen2_single_mount.yaml</parameters>
+			<parameters>$(find ezgripper_control)/config/controllers_single_mount.yaml</parameters>
 		</plugin>
 	</gazebo>

File: ezgripper_description/urdf/ezgripper_single_mount_standalone.urdf.xacro (robot description, xacro)
@@ -1,12 +1,13 @@
 <?xml version="1.0" encoding="UTF-8"?>
-<robot name="ezgripper_dual_gen2_triple_mount" xmlns:xacro="http://ros.org/wiki/xacro">
+<robot name="ezgripper_single_mount" xmlns:xacro="http://ros.org/wiki/xacro">
 	<xacro:property name="ezgripper_offset_x" value="0.02"/>
 	<xacro:property name="ezgripper_offset_y" value="0.0"/>
 	<xacro:property name="ezgripper_offset_z" value="0.3"/>
 	<xacro:include filename="$(find ezgripper_description)/urdf/materials.urdf.xacro"/>
-	<xacro:include filename="$(find ezgripper_description)/urdf/dual_gen2_triple_mount/ezgripper_dual_gen2_triple_mount.urdf.xacro"/>
+	<xacro:include filename="$(find ezgripper_description)/urdf/ezgripper_single_mount.urdf.xacro"/>
 	<!-- Add the gripper -->
-	<xacro:ezgripper_dual_gen2_triple_mount prefix="left" parent_link="base_link"
-			ox="${ezgripper_offset_x}" oy="${ezgripper_offset_y}" oz="${ezgripper_offset_z}"/>
+	<xacro:ezgripper_single_mount prefix="left" parent_link="base_link">
+		<origin xyz="${ezgripper_offset_x} ${ezgripper_offset_y} ${ezgripper_offset_z}" rpy="0 0 0"/>
+	</xacro:ezgripper_single_mount>
 	<link name="world"/>
 	<joint name="fixed" type="fixed">

File: ezgripper_description/urdf/materials.urdf.xacro (robot description, xacro)
@@ -1,4 +1,4 @@
 <?xml version="1.0"?>
-<robot name="ezgripper" xmlns:xacro="http://ros.org/wiki/xacro">
+<robot name="ezgripper_single_mount" xmlns:xacro="http://ros.org/wiki/xacro">
   <material name="black">
     <color rgba="0.0 0.0 0.0 1.0"/>
